File: dispenser_pcb_kicad/_saved_dispenser_pcb_rev01.sch (KiCad schematic (older format))
At the start: 36 parts, among them CON1 BARREL_JACK, IC1 ATMEGA328P-P, P1 RPI_GPIO_HEADER, P10 CONN_01X01, P11 CONN_01X01, P12 CONN_02X03, P2 CONN_01X04, P3 CONN_01X04, P4 CONN_01X03, P5 CONN_01X04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

Commit message: .
Parts:
- C10: renamed from C?; footprint Capacitors_THT:CP_Radial_D6.3mm_P2.50mm -> Capacitors_ThroughHole:C_Radial_D6.3_L11.2_P2.5
- C8: footprint Capacitors_THT:CP_Radial_D6.3mm_P2.50mm -> Capacitors_ThroughHole:C_Radial_D6.3_L11.2_P2.5
- gave numbers to parts that had none: 4
Changed lines of the file:
@@
 $EndComp
 Wire Wire Line
-	7200 2200 7200 2350
-Wire Wire Line
-	7200 2350 7200 2450
-Wire Wire Line
-	7200 2450 7200 2750
+	7200 2200 7200 2750
 Wire Wire Line
 	7200 2450 7300 2450
@@
 	7300 4650 7200 4650
 Wire Wire Line
-	7200 4650 7200 4750
-Wire Wire Line
-	7200 4750 7200 4900
+	7200 4650 7200 4900
 Wire Wire Line
 	7300 4750 7200 4750
@@
 	14150 3550 14050 3550
 Wire Wire Line
-	14050 3550 14050 3650
-Wire Wire Line
-	14050 3650 14050 3750
+	14050 3550 14050 3750
 Wire Wire Line
 	14150 3650 14050 3650
@@
 	14150 1700 14050 1700
 Wire Wire Line
-	14050 1700 14050 1800
-Wire Wire Line
-	14050 1800 14050 1900
+	14050 1700 14050 1900
 Wire Wire Line
 	14150 1800 14050 1800
@@
 	7400 5550 7400 5600
 Wire Wire Line
-	7400 5900 7400 5950
-Wire Wire Line
-	7400 5950 7400 6050
+	7400 5900 7400 6050
 Wire Wire Line
 	7400 6350 7400 6250
@@
 	8650 9600 8650 9500
 Wire Wire Line
-	8650 8500 8650 8750
-Wire Wire Line
-	8650 8750 8650 8900
+	8650 8500 8650 8900
 Wire Wire Line
 	8650 8750 8800 8750
@@
 	8450 8850 8450 8900
 Wire Wire Line
-	7850 9200 7950 9200
-Wire Wire Line
-	7950 9200 8200 9200
+	7850 9200 8200 9200
 Wire Wire Line
 	7950 9200 7950 9300
@@
 Connection ~ 7950 9200
 Wire Wire Line
-	7250 9200 7450 9200
-Wire Wire Line
-	7450 9200 7550 9200
+	7250 9200 7550 9200
 Wire Wire Line
 	7450 9200 7450 9250
@@
 	13400 8600 13500 8600
 Wire Wire Line
-	13500 8600 13500 8700
-Wire Wire Line
-	13500 8700 13500 8850
+	13500 8600 13500 8850
 Wire Wire Line
 	13400 8700 13500 8700
@@
 	3750 2500 3650 2500
 Wire Wire Line
-	3650 2400 3650 2500
-Wire Wire Line
-	3650 2500 3650 2600
+	3650 2400 3650 2600
 Wire Wire Line
 	3650 2600 3750 2600
@@
 	3500 2900 3750 2900
 Wire Wire Line
-	3500 2750 3500 2800
-Wire Wire Line
-	3500 2800 3500 2900
+	3500 2750 3500 2900
 Wire Wire Line
 	3500 2800 3750 2800
@@
 	3750 4300 3600 4300
 Wire Wire Line
-	3600 4300 3600 4400
-Wire Wire Line
-	3600 4400 3600 4500
-Wire Wire Line
-	3600 4500 3600 4600
-Wire Wire Line
-	3600 4600 3600 4700
-Wire Wire Line
-	3600 4700 3600 4800
-Wire Wire Line
-	3600 4800 3600 4900
-Wire Wire Line
-	3600 4900 3600 5000
-Wire Wire Line
-	3600 5000 3600 5200
+	3600 4300 3600 5200
 Wire Wire Line
 	3750 5000 3600 5000
@@
 	11100 4950 11100 5000
 Wire Wire Line
-	10850 4950 10950 4950
-Wire Wire Line
-	10950 4950 11100 4950
+	10850 4950 11100 4950
 Wire Wire Line
 	10950 4950 10950 4850
@@
 	11200 5000 11200 4950
 Wire Wire Line
-	11200 4950 11350 4950
-Wire Wire Line
-	11350 4950 11450 4950
+	11200 4950 11450 4950
 Wire Wire Line
 	11350 4950 11350 4850
@@
 $EndComp
 Wire Wire Line
-	2650 7600 3000 7600
-Wire Wire Line
-	3000 7600 3300 7600
-Wire Wire Line
-	2650 7550 2650 7600
-Wire Wire Line
-	2650 7600 2650 7700
-Wire Wire Line
-	2650 8100 3000 8100
-Wire Wire Line
-	3000 8100 3200 8100
-Wire Wire Line
-	3200 8100 3300 8100
-Wire Wire Line
-	2650 8000 2650 8100
-Wire Wire Line
-	2650 8100 2650 8200
-Wire Wire Line
-	4100 7850 4400 7850
-Wire Wire Line
-	4400 7850 4600 7850
+	2650 7600 3300 7600
+Wire Wire Line
+	2650 7550 2650 7700
+Wire Wire Line
+	2650 8100 3300 8100
+Wire Wire Line
+	2650 8000 2650 8200
+Wire Wire Line
+	4100 7850 4600 7850
 $Comp
 L GND #PWR037
@@
 F 0 "C8" H 2675 7950 50  0000 L CNN
 F 1 "5ZLH100MEFC6.3X11" V 3325 7450 50  0001 L CNN
-F 2 "Capacitors_THT:CP_Radial_D6.3mm_P2.50mm" V 3425 7750 50  0001 C CNN
+F 2 "Capacitors_ThroughHole:C_Radial_D6.3_L11.2_P2.5" V 3425 7750 50  0001 C CNN
 F 3 "" H 2650 7850 50  0000 C CNN
 F 4 "100uF 35V" H 2925 7725 60  0000 C CNN "Field4"
@@
 	7950 5750 7850 5750
 Wire Wire Line
-	7200 5950 7400 5950
-Wire Wire Line
-	7400 5950 7950 5950
+	7200 5950 7950 5950
 Text GLabel 7200 5950 0    50   Input ~ 0
 RESET
@@
 POWER BUDGET (worst case)\nRasberry Pi: 1A\nUSB RFID: 50mA\nDisplay: 500mA(?)\nTotal worst case:\n1550mA\n\nAssuming 80% regulator efficiency, current drawn from the 12V\nline will be about 500mA\n
 Wire Wire Line
-	4800 7850 5000 7850
-Wire Wire Line
-	5000 7850 5300 7850
-$Comp
-L LM2576SX U?
+	4800 7850 5300 7850
+$Comp
+L LM2576SX U5
 U 1 1 5B313611
 P 3700 7850
-F 0 "U?" H 3700 8300 60  0000 C CNN
+F 0 "U5" H 3700 8300 60  0000 C CNN
 F 1 "LM2576SX" H 3700 7400 60  0000 C CNN
 F 2 "TO_SOT_Packages_SMD:TO-263-5Lead" H 3700 8400 60  0001 C CNN
@@
 Connection ~ 3200 8100
 $Comp
-L GND #PWR?
+L GND #PWR040
 U 1 1 5B314410
 P 4200 8500
-F 0 "#PWR?" H 4200 8250 50  0001 C CNN
+F 0 "#PWR040" H 4200 8250 50  0001 C CNN
 F 1 "GND" H 4200 8350 50  0000 C CNN
 F 2 "" H 4200 8500 50  0000 C CNN
@@
 $EndComp
 Wire Wire Line
-	4200 8100 4200 8350
-Wire Wire Line
-	4200 8350 4200 8500
+	4200 8100 4200 8500
 Wire Wire Line
 	4200 8100 4100 8100
 Wire Wire Line
-	5000 7500 5000 7600
-Wire Wire Line
-	5000 7600 5000 7850
-Wire Wire Line
-	5000 7850 5000 7950
+	5000 7500 5000 7950
 Wire Wire Line
 	5000 7600 4100 7600
 Wire Wire Line
-	4200 8350 4400 8350
-Wire Wire Line
-	4400 8350 5000 8350
-Wire Wire Line
-	5000 8350 5300 8350
+	4200 8350 5300 8350
 Wire Wire Line
 	4400 8350 4400 8200
@@
 Connection ~ 4400 7850
 $Comp
-L 5ZLH100MEFC6.3X11 C?
+L 5ZLH100MEFC6.3X11 C10
 U 1 1 5B314FC1
 P 5000 8100
-F 0 "C?" H 5025 8200 50  0000 L CNN
+F 0 "C10" H 5025 8200 50  0000 L CNN
 F 1 "5ZLH100MEFC6.3X11" V 5675 7700 50  0001 L CNN
-F 2 "Capacitors_THT:CP_Radial_D6.3mm_P2.50mm" V 5775 8000 50  0001 C CNN
+F 2 "Capacitors_ThroughHole:C_Radial_D6.3_L11.2_P2.5" V 5775 8000 50  0001 C CNN
 F 3 "" H 5000 8100 50  0000 C CNN
 F 4 "100uF 35V" H 4950 7700 60  0000 C CNN "Field4"
@@
 $EndComp
 $Comp
-L C_Small C?
+L C_Small C11
 U 1 1 5B314FC7
 P 5300 8100
-F 0 "C?" H 5310 8170 50  0000 L CNN
+F 0 "C11" H 5310 8170 50  0000 L CNN
 F 1 "0.1uF" H 5050 8150 50  0000 L CNN
 F 2 "Capacitors_SMD:C_0805_HandSoldering" H 5300 8100 50  0001 C CNN
@@
 	5300 7850 5300 8000
 $Comp
-L +5V #PWR?
+L +5V #PWR041
 U 1 1 5B3155F4
 P 5000 7500
-F 0 "#PWR?" H 5000 7350 50  0001 C CNN
+F 0 "#PWR041" H 5000 7350 50  0001 C CNN
 F 1 "+5V" H 5000 7640 50  0000 C CNN
 F 2 "" H 5000 7500 50  0000 C CNN
@@
 Connection ~ 5000 8350
 $Comp
-L B560C-13-F D?
+L B560C-13-F D1
 U 1 1 5B316EE7
 P 4400 8050
-F 0 "D?" H 4400 8150 50  0000 C CNN
+F 0 "D1" H 4400 8150 50  0000 C CNN
 F 1 "B560C-13-F" H 4450 7950 50  0000 C CNN
 F 2 "Diodes_SMD:SMC_Standard" H 4400 8050 50  0001 C CNN
@@
 $EndComp
 $Comp
-L PA4309.104NLT L?
+L PA4309.104NLT L1
 U 1 1 5B3178CA
 P 4700 7850
-F 0 "L?" V 4800 7950 50  0000 L CNN
+F 0 "L1" V 4800 7950 50  0000 L CNN
 F 1 "PA4309.104NLT" H 5000 7850 50  0001 L CNN
 F 2 "USER_INDUCTORS:PA4309.104NLT" H 5600 7800 50  0001 C CNN
