File: dispenser_pcb_kicad/dispenser_pcb_rev01.kicad_pcb (KiCad board)
At the start: 2 copper layers, 150.5 x 85.7 mm, 28 parts, among them CON1 BARREL_JACK, IC1 ATMEGA328P-P, P1 RPI_GPIO_HEADER, P10 CONN_01X01, P11 CONN_01X01, P2 CONN_01X04, P3 CONN_01X04, P4 CONN_01X03, P5 CONN_01X04, P6 CONN_01X04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

Commit message: cc
Parts:
- added C8: 5ZLH100MEFC6.3X11, Capacitors_THT:CP_Radial_D6.3mm_P2.50mm, F.Cu at (130.8, 57.9)
- added C9: 0.1uF, Capacitors_SMD:C_0805_HandSoldering, F.Cu at (131.8, 52.8)
- added P12: CONN_02X03, Pin_Headers:Pin_Header_Straight_2x03_Pitch2.54mm, F.Cu at (198.1, 56.9)
- moved C3 46.0 mm to (178.3, 98.3)
- moved C5 46.0 mm to (178.3, 90.7)
- moved R2 46.0 mm to (184.7, 94.5)
- moved C4 46.0 mm to (183.4, 90.7)
- moved R3 46.0 mm to (183.4, 98.3)
- moved U3 46.0 mm to (181.0, 94.5)
- moved C1 45.0 mm to (190.5, 73.7), turned to 270 degrees
- moved R4 44.9 mm to (196.9, 83.8), turned to 180 degrees
- moved P4 44.5 mm to (163.9, 108.0)
- moved C7 43.0 mm to (196.9, 78.7), turned to 0 degrees
- moved R1 39.6 mm to (177.8, 73.6), turned to 90 degrees
- moved C2 39.5 mm to (175.3, 73.7), turned to 90 degrees
- moved U4 35.2 mm to (190.6, 81.2), turned to 270 degrees
- moved IC1 34.1 mm to (175.3, 69.8), turned to 90 degrees
- moved P6 29.2 mm to (191.8, 108.0)
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Connections:
- net M2_DIR renamed M2_DIR(MOSI)
- net Net-(C2-Pad2) renamed RESET
- IC1 pad 18: Net-(IC1-Pad18) -> MISO
- IC1 pad 19: Net-(IC1-Pad19) -> SCK
Routing:
- net +12V: track 0.00 -> 166.2 mm
- net RESET: track 0.00 -> 43.3 mm
- net TX: track 0.00 -> 34.7 mm
- net RX: track 0.00 -> 27.0 mm
- net +3V3: track 0.00 -> 15.1 mm
- net Net-(IC1-Pad5): track 0.00 -> 14.0 mm
- net MISO: track 0.00 -> 11.3 mm
- net STEPPER1_2B: track 0.00 -> 9.86 mm
- net STEPPER1_2A: track 0.00 -> 9.85 mm
- net STEPPER1_1A: track 0.00 -> 9.83 mm
- net LOADCELL+: track 0.00 -> 9.82 mm
- net STEPPER1_1B: track 0.00 -> 9.81 mm
- net Net-(IC1-Pad6): track 0.00 -> 9.35 mm
- net M2_DIR(MOSI): track 0.00 -> 8.93 mm
- net STEPPER2_1B: track 0.00 -> 8.06 mm
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- added copper zone on B.Cu, net GND
- added copper zone on F.Cu, net GND

Commit message: .
Parts:
- added C10: 5ZLH100MEFC6.3X11, Capacitors_ThroughHole:C_Radial_D6.3_L11.2_P2.5, F.Cu at (162.1, 148.8)
- added C11: 0.1uF, Capacitors_SMD:C_0805_HandSoldering, F.Cu at (159.5, 143.8)
- added D1: B560C-13-F, Diodes_SMD:SMC_Standard, F.Cu at (141.2, 150.4)
- added L1: PA4309.104NLT, USER_INDUCTORS:PA4309.104NLT, F.Cu at (152.7, 153.4)
- added U5: LM2576SX, TO_SOT_Packages_SMD:TO-263-5Lead, F.Cu at (152.9, 143.5)
- C8: footprint Capacitors_THT:CP_Radial_D6.3mm_P2.50mm -> Capacitors_ThroughHole:C_Radial_D6.3_L11.2_P2.5
- moved U2 141.0 mm to (275.6, 102.9), turned to 180 degrees
- moved U1 138.0 mm to (294.1, 102.9), turned to 180 degrees
- moved C9 92.1 mm to (146.3, 143.8), turned to 270 degrees
- moved C8 84.7 mm to (143.0, 141.7), turned to 180 degrees
- moved CON1 73.1 mm to (128.5, 112.2), turned to 90 degrees
- moved C2 51.3 mm to (223.5, 56.4)
- moved C3 51.3 mm to (226.6, 81.0)
- moved C5 51.3 mm to (226.6, 73.4)
- moved C7 51.3 mm to (245.2, 61.4)
- moved IC1 51.3 mm to (223.5, 52.6)
- moved R2 51.3 mm to (232.9, 77.2)
- moved R4 51.3 mm to (245.2, 66.5)
- moved R3 51.3 mm to (231.6, 81.0)
- moved U4 51.3 mm to (238.8, 64.0)
- moved C1 51.3 mm to (238.8, 56.4)
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Routing:
- net +12V: track 166.2 -> 0.00 mm
- net TX: track 34.7 -> 4.67 mm
- net RX: track 27.0 -> 3.56 mm
- net STEPPER1_2B: track 9.86 -> 0.00 mm
- net STEPPER1_2A: track 9.85 -> 0.00 mm
- net STEPPER1_1A: track 9.83 -> 0.00 mm
- net LOADCELL+: track 9.82 -> 0.00 mm
- net STEPPER1_1B: track 9.81 -> 0.00 mm
- net STEPPER2_1B: track 8.06 -> 0.00 mm
- net STEPPER2_1A: track 8.04 -> 0.00 mm
- net STEPPER2_2A: track 8.02 -> 0.00 mm
- net STEPPER2_2B: track 8.01 -> 0.00 mm
- net LOADCELL-: track 7.64 -> 0.00 mm
- net Net-(IC1-Pad6): track 9.35 -> 2.77 mm
- net STRIP2_DATA: track 6.15 -> 0.00 mm
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- added copper zone on F.Cu, net +12V
- added copper zone on F.Cu, net +5V
- added copper zone on F.Cu, net Net-(D1-Pad1)
