File: dispenser_pcb_kicad/dispenser_pcb_rev01.sch (KiCad schematic (older format))
At the start: 28 parts, among them CON1 BARREL_JACK, IC1 ATMEGA328P-P, P1 RPI_GPIO_HEADER, P10 CONN_01X01, P11 CONN_01X01, P2 CONN_01X04, P3 CONN_01X04, P4 CONN_01X03, P5 CONN_01X04, P6 CONN_01X04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

Commit message: cc
Parts:
- added C8: 5ZLH100MEFC6.3X11, Capacitors_THT:CP_Radial_D6.3mm_P2.50mm, symbol 5ZLH100MEFC6.3X11
- added C9: 0.1uF, Capacitors_SMD:C_0805_HandSoldering, symbol C_Small
- added L1: L_s, symbol L_s
- added P12: CONN_02X03, Pin_Headers:Pin_Header_Straight_2x03_Pitch2.54mm, symbol CONN_02X03
Connections:
- net +12V: now also C8.1, C9.1
- net +3V3: now also P12.2 (P2)
- net GND: now also C8.2, C9.2, P12.6 (P6)
- net RESET: now reaches C2.2, IC1.1 ((PCINT14/~RESET~)PC6), R1.2
- net RESET: now also P12.5 (P5)
- net MISO: now reaches IC1.18 ((PCINT4/MISO)PB4)
- net MISO: now also P12.1 (P1)
- net SCK: now reaches IC1.19 ((PCINT5/SCK)PB5)
- net SCK: now also P12.3 (P3)
- net M2_DIR renamed M2_DIR(MOSI)
- net M2_DIR(MOSI): now also P12.4 (P4)
Other:
- note added: "PROGRAMMING HEADER"
- moved on the sheet: C2, R1

Commit message: .
Parts:
- removed L1: L_s, symbol L_s
- added C10: 5ZLH100MEFC6.3X11, Capacitors_THT:CP_Radial_D6.3mm_P2.50mm, symbol 5ZLH100MEFC6.3X11
- added C11: 0.1uF, Capacitors_SMD:C_0805_HandSoldering, symbol C_Small
- added D1: B560C-13-F, Diodes_SMD:SMC_Standard, symbol B560C-13-F
- added L1: PA4309.104NLT, USER_INDUCTORS:PA4309.104NLT, symbol PA4309.104NLT
- added U5: LM2576SX, TO_SOT_Packages_SMD:TO-263-5Lead, symbol LM2576SX
Connections:
- net +12V: now also U5.1 (VIN)
- net +5V: now also C10.1, C11.1, L1.2, U5.4 (FB)
- net GND: now also C10.2, C11.2, D1.2 (A), U5.3 (TGND), U5.5 (ON/OFF)
- new net: D1.1 (K), L1.1, U5.2 (OUT)
Other:
- note added: "POWER BUDGET (worst case)\nRasberry Pi: 1A\nUSB RFID: 50mA\nDisplay: 500mA(?)\nTotal worst case:\n1550mA\n\nAssuming 80% regulator efficiency, current drawn from the 12V\nline will be about 500mA\n"
- moved on the sheet: C8, C9, P10, P11, P8, P9
